Commit message: Add camera to phantomx and change physics engine

File: mara_description/urdf/phantomx.urdf (robot description, URDF)
Before this commit: robot PhantomX, 26 links, 25 joints
Links:
- added link camera_link, mass 0
- link MP_BODY: mass 1.97559947 -> 1.0
Joints:
- added joint camera_joint: type fixed, parent MP_BODY, child camera_link, origin xyz=0 -0.6 0.5 rpy=0 0.8 1.5708, axis 0 1 0
- joint j_phantomx_attachment: origin xyz=0 0 0 rpy=0 0 0 -> xyz=0 0 0.3 rpy=0 0 0
- joint j_thigh_lf: limit lower=-1.5708 upper=1.5708 effort=2.8 velocity=5.6548668 -> lower=-1.3 upper=-0.3 effort=2.8 velocity=5.6548668
- joint j_thigh_lm: limit lower=-1.5708 upper=1.5708 effort=2.8 velocity=5.6548668 -> lower=-1.3 upper=-0.3 effort=2.8 velocity=5.6548668
- joint j_thigh_lr: limit lower=-1.5708 upper=1.5708 effort=2.8 velocity=5.6548668 -> lower=-1.3 upper=-0.3 effort=2.8 velocity=5.6548668
- joint j_thigh_rf: limit lower=-1.5708 upper=1.5708 effort=2.8 velocity=5.6548668 -> lower=-1.3 upper=-0.3 effort=2.8 velocity=5.6548668
- joint j_thigh_rm: limit lower=-1.5708 upper=1.5708 effort=2.8 velocity=5.6548668 -> lower=-1.3 upper=-0.3 effort=2.8 velocity=5.6548668
- joint j_thigh_rr: limit lower=-1.5708 upper=1.5708 effort=2.8 velocity=5.6548668 -> lower=-1.3 upper=-0.3 effort=2.8 velocity=5.6548668
- joint j_tibia_lf: limit lower=-2.53073 upper=0.6179939 effort=2.8 velocity=5.6548668 -> lower=-2.0 upper=-1.5 effort=2.8 velocity=5.6548668
- joint j_tibia_lm: limit lower=-2.53073 upper=0.6179939 effort=2.8 velocity=5.6548668 -> lower=-2.0 upper=-1.5 effort=2.8 velocity=5.6548668
- joint j_tibia_lr: limit lower=-2.53073 upper=0.6179939 effort=2.8 velocity=5.6548668 -> lower=-2.0 upper=-1.5 effort=2.8 velocity=5.6548668
- joint j_tibia_rf: limit lower=-2.53073 upper=0.6179939 effort=2.8 velocity=5.6548668 -> lower=-2.0 upper=-1.5 effort=2.8 velocity=5.6548668
- joint j_tibia_rm: limit lower=-2.53073 upper=0.6179939 effort=2.8 velocity=5.6548668 -> lower=-2.0 upper=-1.5 effort=2.8 velocity=5.6548668
- joint j_tibia_rr: limit lower=-2.53073 upper=0.6179939 effort=2.8 velocity=5.6548668 -> lower=-2.0 upper=-1.5 effort=2.8 velocity=5.6548668

Commit message: Changes in spawn phantomx

File: mara_description/urdf/phantomx.urdf (robot description, URDF)
Before this commit: robot PhantomX, 27 links, 26 joints
Joints:
- joint j_phantomx_attachment: origin xyz=0 0 0.3 rpy=0 0 0 -> xyz=0 0 0 rpy=0 0 0
